File: RF-input-bandpass.brd (EAGLE design)
At the start: 30 x 29 mm, 8 parts, among them J2 DC 0 AC 1E-6

Commit message: Update trace clearance, add corner holes
Routing:
- net 0: track 58.9 -> 0.00 mm
- net N$2: track 41.4 -> 50.1 mm
- net N$3: track 5.98 -> 11.5 mm, vias 0 -> 1
- net N$6: track 5.41 -> 0.00 mm, vias 1 -> 0
- net N$5: track 2.00 -> 0.00 mm, vias 1 -> 0
- net N$4: track 18.9 -> 19.8 mm
- added copper zone on layer 16, net 0
- removed copper zone on layer 16, net GND
Other:
- board text removed: "GND"

Commit message: Increase trace and clearance size
Routing:
- net N$4: track 19.8 -> 40.2 mm
- net N$2: track 50.1 -> 43.6 mm
- net N$1: track 12.9 -> 17.2 mm
- net N$3: track 11.5 -> 8.43 mm

Commit message: Add missing R1 to brd, invert layout png colors
Parts:
- added R1: 68, adafruit:0204V
Connections:
- net 0: now also R1.1
- net N$4: now also R1.2
Routing:
- net 0: track 0.00 -> 0.73 mm
Changed lines of the file:
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@@
 <grid distance="1" unitdist="mm" unit="mm" style="lines" multiple="1" display="no" altdistance="0.1" altunitdist="mil" altunit="mm"/>
 <layers>
-<layer number="1" name="Top" color="4" fill="1" visible="no" active="yes"/>
+<layer number="1" name="Top" color="4" fill="1" visible="yes" active="yes"/>
 <layer number="16" name="Bottom" color="1" fill="1" visible="yes" active="yes"/>
 <layer number="17" name="Pads" color="2" fill="1" visible="yes" active="yes"/>
 <layer number="18" name="Vias" color="2" fill="1" visible="yes" active="yes"/>
-<layer number="19" name="Unrouted" color="6" fill="1" visible="no" active="yes"/>
-<layer number="20" name="Dimension" color="24" fill="1" visible="no" active="yes"/>
-<layer number="21" name="tPlace" color="7" fill="1" visible="no" active="yes"/>
-<layer number="22" name="bPlace" color="7" fill="1" visible="no" active="yes"/>
-<layer number="23" name="tOrigins" color="15" fill="1" visible="no" active="yes"/>
-<layer number="24" name="bOrigins" color="15" fill="1" visible="no" active="yes"/>
-<layer number="25" name="tNames" color="7" fill="1" visible="no" active="yes"/>
-<layer number="26" name="bNames" color="7" fill="1" visible="no" active="yes"/>
-<layer number="27" name="tValues" color="7" fill="1" visible="no" active="yes"/>
+<layer number="19" name="Unrouted" color="6" fill="1" visible="yes" active="yes"/>
+<layer number="20" name="Dimension" color="24" fill="1" visible="yes" active="yes"/>
+<layer number="21" name="tPlace" color="7" fill="1" visible="yes" active="yes"/>
+<layer number="22" name="bPlace" color="7" fill="1" visible="yes" active="yes"/>
+<layer number="23" name="tOrigins" color="15" fill="1" visible="yes" active="yes"/>
+<layer number="24" name="bOrigins" color="15" fill="1" visible="yes" active="yes"/>
+<layer number="25" name="tNames" color="7" fill="1" visible="yes" active="yes"/>
+<layer number="26" name="bNames" color="7" fill="1" visible="yes" active="yes"/>
+<layer number="27" name="tValues" color="7" fill="1" visible="yes" active="yes"/>
 <layer number="28" name="bValues" color="7" fill="1" visible="no" active="yes"/>
 <layer number="29" name="tStop" color="7" fill="3" visible="no" active="yes"/>
@@
 <attribute name="SPICEPREFIX" value="L" x="-20.67" y="-9.75" size="1.778" layer="27" rot="R270" display="off"/>
 </element>
+<element name="R1" library="adafruit" library_urn="urn:adsk.eagle:library:420" package="0204V" package3d_urn="urn:adsk.eagle:package:6240630/1" value="68" x="25.083259375" y="16.532359375" smashed="yes" rot="R180">
+<attribute name="NAME" x="26.216859375" y="18.363959375" size="1.27" layer="25" ratio="12" rot="R180"/>
+<attribute name="SPICEPREFIX" value="R" x="25.083259375" y="16.532359375" size="1.778" layer="27" rot="R180" display="off"/>
+</element>
 </elements>
 <signals>
@@
 <contactref element="L2" pad="2"/>
 <contactref element="C5" pad="1"/>
-<wire x1="23.75" y1="10.25" x2="23.75" y2="19" width="1.016" layer="16"/>
+<wire x1="23.75" y1="10.25" x2="23.75" y2="16" width="1.016" layer="16"/>
+<wire x1="23.75" y1="16.532359375" x2="23.75" y2="19" width="1.016" layer="16"/>
 <wire x1="24" y1="10.25" x2="23.75" y2="10.25" width="1.016" layer="16"/>
 <wire x1="25.25" y1="9" x2="24" y2="10.25" width="1.016" layer="16"/>
@@
 <wire x1="15" y1="10.75" x2="20.75" y2="5" width="1.016" layer="16"/>
 <wire x1="15" y1="11" x2="15" y2="10.75" width="1.016" layer="16"/>
-<wire x1="6.5" y1="19.5" x2="15" y2="11" width="1.016" layer="16"/>
+<wire x1="6.5" y1="19.5" x2="12.4539" y2="13.5461" width="1.016" layer="16"/>
+<wire x1="12.4539" y1="13.5461" x2="15" y2="11" width="1.016" layer="16"/>
 <wire x1="6" y1="19.5" x2="6.5" y2="19.5" width="1.016" layer="16"/>
 <wire x1="23.75" y1="19" x2="23.73" y2="19" width="1.016" layer="16"/>
 <wire x1="6" y1="19.5" x2="6" y2="19.46" width="1.016" layer="16"/>
+<contactref element="R1" pad="2"/>
+<wire x1="23.813259375" y1="16.532359375" x2="23.75" y2="16.532359375" width="1.016" layer="16"/>
+<wire x1="23.75" y1="16.532359375" x2="23.75" y2="16" width="1.016" layer="16"/>
 </signal>
-<signal name="0">
+<signal name="0" airwireshidden="yes">
 <contactref element="C5" pad="2"/>
 <contactref element="J2" pad="2"/>
@@
 <vertex x="0" y="0"/>
 </polygon>
-<wire x1="16.92" y1="13.08" x2="14.27" y2="19" width="0" layer="19" extent="1-1"/>
+<contactref element="R1" pad="1"/>
+<wire x1="14.27" y1="19" x2="15" y2="19" width="1.016" layer="16"/>
+<wire x1="15" y1="19" x2="16.92" y2="13.08" width="0" layer="19" extent="16-16"/>
 </signal>
 </signals>
@@
 <mfgpreviewcolor name="substratecolor" color="0xFF786E46"/>
 </mfgpreviewcolors>
+<errors>
+</errors>
 </board>
 </drawing>
